File: board/chrimbus2019/chrimbus2019.kicad_pcb (KiCad board)
At the start: 2 copper layers, 85.4 x 94.6 mm, 6 parts, among them J1 Conn_01x06, U1 TLC59116F, U2 XC9142, U3 PIC16F15325

Commit message: pre sleep mode
Parts:
- added C1: 0.1uF, Capacitor_SMD:C_0805_2012Metric, F.Cu at (155.0, 75.1)
- added C2: 0.1uF, Capacitor_SMD:C_0805_2012Metric, F.Cu at (148.0, 76.6)
- added C3: 0.1uF, Capacitor_SMD:C_0805_2012Metric, F.Cu at (163.0, 79.3)
- added C4: 10uF, Capacitor_SMD:C_0805_2012Metric, F.Cu at (142.9, 75.0)
- added D1: LED, toolbox_LED:LTST-C150AKT, F.Cu at (133.5, 79.8)
- added D10: LED, toolbox_LED:LTST-C150AKT, F.Cu at (177.2, 79.6)
- added D11: LED, toolbox_LED:LTST-C150AKT, F.Cu at (186.6, 68.1)
- added D12: LED, toolbox_LED:LTST-C150AKT, F.Cu at (180.8, 57.1)
- added D13: LED, toolbox_LED:LTST-C150AKT, F.Cu at (165.5, 61.0)
- added D14: LED, toolbox_LED:LTST-C150AKT, F.Cu at (144.1, 61.0)
- added D15: LED, toolbox_LED:LTST-C150AKT, F.Cu at (128.8, 58.2)
- added D16: LED, toolbox_LED:LTST-C150AKT, F.Cu at (122.6, 68.2)
- added D2: LED, toolbox_LED:LTST-C150AKT, F.Cu at (124.3, 91.8)
- added D3: LED, toolbox_LED:LTST-C150AKT, F.Cu at (128.7, 101.4)
- added D4: LED, toolbox_LED:LTST-C150AKT, F.Cu at (143.8, 98.5)
- added D5: LED, toolbox_LED:LTST-C150AKT, F.Cu at (148.8, 113.4)
- added D6: LED, toolbox_LED:LTST-C150AKT, F.Cu at (160.5, 113.5)
- added D7: LED, toolbox_LED:LTST-C150AKT, F.Cu at (166.2, 99.3)
- added D8: LED, toolbox_LED:LTST-C150AKT, F.Cu at (180.8, 101.2)
- added D9: LED, toolbox_LED:LTST-C150AKT, F.Cu at (187.1, 90.9)
- added L1: 4.7uH, Inductor_SMD:L_0805_2012Metric, F.Cu at (139.3, 77.0)
- added R1: 10k, Resistor_SMD:R_0603_1608Metric, F.Cu at (158.7, 73.5)
- added R10: 150, Resistor_SMD:R_0603_1608Metric, F.Cu at (183.9, 91.7)
- added R11: 150, Resistor_SMD:R_0603_1608Metric, F.Cu at (174.0, 79.5)
- added R12: 150, Resistor_SMD:R_0603_1608Metric, F.Cu at (183.5, 67.3)
- added R13: 150, Resistor_SMD:R_0603_1608Metric, F.Cu at (179.9, 60.2)
- added R14: 150, Resistor_SMD:R_0603_1608Metric, F.Cu at (163.9, 63.8)
- added R15: 150, Resistor_SMD:R_0603_1608Metric, F.Cu at (145.7, 63.7)
- added R16: 150, Resistor_SMD:R_0603_1608Metric, F.Cu at (129.8, 61.4)
- added R17: 150, Resistor_SMD:R_0603_1608Metric, F.Cu at (125.9, 67.3)
- added R18: 150, Resistor_SMD:R_0603_1608Metric, F.Cu at (165.6, 84.7)
- added R19: 10K, Resistor_SMD:R_0603_1608Metric, F.Cu at (156.3, 90.2)
- added R2: 150, Resistor_SMD:R_0603_1608Metric, F.Cu at (136.6, 79.7)
- added R20: 10k, Resistor_SMD:R_0603_1608Metric, F.Cu at (168.2, 85.5)
- added R21: 10k, Resistor_SMD:R_0603_1608Metric, F.Cu at (168.6, 70.1)
- added R22: 10k, Resistor_SMD:R_0603_1608Metric, F.Cu at (166.8, 70.1)
- added R3: 150, Resistor_SMD:R_0603_1608Metric, F.Cu at (127.6, 92.8)
- added R4: 150, Resistor_SMD:R_0603_1608Metric, F.Cu at (129.7, 98.1)
- added R5: 150, Resistor_SMD:R_0603_1608Metric, F.Cu at (145.6, 95.5)
- added R6: 150, Resistor_SMD:R_0603_1608Metric, F.Cu at (151.0, 111.2)
- added R7: 150, Resistor_SMD:R_0603_1608Metric, F.Cu at (158.4, 111.4)
- added R8: 150, Resistor_SMD:R_0603_1608Metric, F.Cu at (164.8, 96.7)
- added R9: 150, Resistor_SMD:R_0603_1608Metric, F.Cu at (180.0, 98.2)
- added SW1: SW_Push, toolbox_switch:TL3305AF160QG, F.Cu at (155.2, 93.5)
- added TP1: TestPoint, TestPoint:TestPoint_Keystone_5000-5004_Miniature, F.Cu at (177.5, 66.7)
- added TP2: TestPoint, TestPoint:TestPoint_Keystone_5000-5004_Miniature, F.Cu at (166.2, 65.0)
- BT1: value Battery_Cell -> CR2450; footprint Battery:BatteryHolder_Keystone_103_1x20mm -> toolbox_battery:BAT_BK-877
- MH1: footprint MountingHole:MountingHole_2.5mm -> MountingHole:MountingHole_2.2mm_M2
- U1: footprint Package_SO:SOIC-28W_7.5x17.9mm_P1.27mm -> Package_SO:TSSOP-28_4.4x9.7mm_P0.65mm
- U2: footprint Package_SO:TSOP-5_1.65x3.05mm_P0.95mm -> Package_TO_SOT_SMD:SOT-23-5_HandSoldering
- U3: footprint Package_SO:SOIC-14_3.9x8.7mm_P1.27mm -> Package_SO:TSSOP-14_4.4x5mm_P0.65mm
- moved J1 29.4 mm to (152.0, 63.5)
- moved U2 25.3 mm to (143.1, 78.6), turned to 180 degrees
- moved U3 22.4 mm to (166.9, 79.3), turned to 90 degrees
- moved BT1 13.5 mm to (154.9, 79.0), turned to 180 degrees
- moved MH1 9.05 mm to (154.9, 37.1)
- moved U1 7.63 mm to (154.9, 81.4)
Connections:
- BT1 pad 1: Net-(BT1-Pad1) -> +BATT
- BT1 pad 2: Net-(BT1-Pad2) -> GND
- J1 pad 1: Net-(J1-Pad1) -> /MCLR
- J1 pad 2: Net-(J1-Pad2) -> +3V3
- J1 pad 3: Net-(J1-Pad3) -> GND
- J1 pad 4: Net-(J1-Pad4) -> /ICSPD
- J1 pad 5: Net-(J1-Pad5) -> /ICSPC
- U1 pad 10: Net-(U1-Pad10) -> GND
- U1 pad 19: Net-(U1-Pad19) -> GND
- U1 pad 2: Net-(U1-Pad2) -> GND
- U1 pad 24: Net-(U1-Pad24) -> GND
- U1 pad 26: Net-(U1-Pad26) -> /SCL
- U1 pad 27: Net-(U1-Pad27) -> /SDA
- U1 pad 28: Net-(U1-Pad28) -> +3V3
- U1 pad 3: Net-(U1-Pad3) -> GND
- U1 pad 4: Net-(U1-Pad4) -> GND
- U1 pad 5: Net-(U1-Pad5) -> GND
- U2 pad 1: Net-(U2-Pad1) -> /CE
- U2 pad 2: Net-(U2-Pad2) -> GND
- U2 pad 3: Net-(U2-Pad3) -> +BATT
- U2 pad 4: Net-(U2-Pad4) -> +3V3
- U3 pad 1: Net-(U3-Pad1) -> +BATT
- U3 pad 10: Net-(U3-Pad10) -> /SCL
- U3 pad 12: Net-(U3-Pad12) -> /ICSPC
- U3 pad 13: Net-(U3-Pad13) -> /ICSPD
- U3 pad 14: Net-(U3-Pad14) -> GND
- U3 pad 4: Net-(U3-Pad4) -> /MCLR
- U3 pad 6: Net-(U3-Pad6) -> /CE
- U3 pad 9: Net-(U3-Pad9) -> /SDA
Routing:
- net +BATT: track 0.00 -> 61.8 mm, vias 0 -> 6
- net GND: track 0.00 -> 56.1 mm, vias 0 -> 10
- net +3V3: track 0.00 -> 55.3 mm, vias 0 -> 14
- net Net-(R12-Pad2): track 0.00 -> 47.6 mm
- net Net-(R16-Pad2): track 0.00 -> 47.0 mm
- net Net-(R17-Pad2): track 0.00 -> 46.7 mm
- net Net-(R13-Pad2): track 0.00 -> 46.5 mm
- net Net-(R9-Pad2): track 0.00 -> 41.7 mm
- net /MCLR: track 0.00 -> 41.1 mm, vias 0 -> 2
- net Net-(R6-Pad2): track 0.00 -> 38.6 mm
- net Net-(R7-Pad2): track 0.00 -> 38.5 mm
- net Net-(R15-Pad2): track 0.00 -> 33.2 mm
- net /CE: track 0.00 -> 30.8 mm, vias 0 -> 2
- net /SDA: track 0.00 -> 29.9 mm, vias 0 -> 3
- net Net-(R4-Pad2): track 0.00 -> 29.5 mm
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- added copper zone on F.Cu, net +3V3
- added copper zone on B.Cu, net GND
Other:
- board text added: "*"
- board text added: "2019"
- board text added: "LOVE, JAKE"
- board text added: "MERRY CHRISTMAS!"
- board text added: "REV 1"
